File: AS5600-Encoder-PCB.kicad_pcb (KiCad board)
At the start: 2 copper layers, 26 x 17.1 mm, 13 parts, among them IC1 AS5600-ASOM, J1 Conn_01x04_Male, J2 Conn_01x04_Male

Commit message: Fixed .gitignore
Parts:
- removed REF**: MountingHole_2.2mm_M2, MountingHole:MountingHole_2.2mm_M2
Changed lines of the file:
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@@
     (tracks 49)
     (zones 0)
-    (modules 13)
+    (modules 12)
     (nets 8)
   )
@@
     (add_net GND)
   )
-  (module MountingHole:MountingHole_2.2mm_M2 (layer F.Cu)
-    (at 188.65 143.77)
-    (descr "Mounting Hole 2.2mm, no annular, M2")
-    (tags "mounting hole 2.2mm no annular m2")
-    (attr virtual)
-    (fp_text reference REF** (at 0 -3.2) (layer F.SilkS)
-      (effects (font (size 1 1) (thickness 0.15)))
-    )
-    (fp_text value MountingHole_2.2mm_M2 (at 0 3.2) (layer F.Fab)
-      (effects (font (size 1 1) (thickness 0.15)))
-    )
-    (fp_circle (center 0 0) (end 2.45 0) (layer F.CrtYd) (width 0.05))
-    (fp_circle (center 0 0) (end 2.2 0) (layer Cmts.User) (width 0.15))
-    (fp_text user %R (at 0.3 0) (layer F.Fab)
-      (effects (font (size 1 1) (thickness 0.15)))
-    )
-    (pad 1 np_thru_hole circle (at 0 0) (size 2.2 2.2) (drill 2.2) (layers *.Cu *.Mask))
-  )
   (module Resistor_THT:R_Axial_DIN0207_L6.3mm_D2.5mm_P10.16mm_Horizontal (layer F.Cu)
